File: LED_Matrix_Phone_Case.kicad_sch (KiCad schematic)
At the start: 608 parts, among them J1 USB_C_PC_Receptacle_F, M1 MountingHole_Pad, M2 MountingHole_Pad, M3 MountingHole_Pad, M4 MountingHole_Pad, P1 USB_C_PhonePlug_M, U2 TPS7A0233PDQNR_PHONE, U3 STM32WB55RGV6, U4 TPS7A0233PDQNR_PC, X1 32.768KHz, X2 32MHz

Commit message: ver 1.1 files, i fucked up the flex board to main board pads on v1.0 but fixed in 1.1
Parts:
- removed C14, C8: 100nF, symbol Device:C_Small
- removed C2, C3: 4.7uF, Capacitor_SMD:C_0603_1608Metric, symbol Device:C_Small
- removed C4: 4.7µF, symbol Device:C_Small
- removed C6: 4.7µF, Capacitor_SMD:C_0603_1608Metric, symbol Device:C_Small
- removed C9: 4.7uF, symbol Device:C_Small
- removed D593, D594, D595, D596, D597, D598, D599, D600, D601, D602, D603, D604: LED, symbol Device:LED
- removed J1: USB_C_PC_Receptacle_F, symbol Connector:USB_C_Receptacle
- removed P1: USB_C_PhonePlug_M, symbol Connector:USB_C_Plug
- removed R1, R2: 5.1kΩ, symbol Device:R_Small_US
- removed R41: 5.1kΩ, Resistor_SMD:R_0603_1608Metric, symbol Device:R_Small_US
- removed U2: TPS7A0233PDQNR_PHONE, TPS7A0233PDQNR:IC_TPS7A0233PDQNR, symbol TPS7A0233PDQNR:TPS7A0233PDQNR
- removed U4: TPS7A0233PDQNR_PC, TPS7A0233PDQNR:IC_TPS7A0233PDQNR, symbol TPS7A0233PDQNR:TPS7A0233PDQNR
- added C17, C18, C7: 4.7uF, Capacitor_SMD:C_0603_1608Metric, symbol Device:C_Small
- added R_NOT_POPULATED1, Rn1, Rn2, Rn3: 0.0Ω, Resistor_SMD:R_0603_1608Metric_Pad0.98x0.95mm_HandSolder, symbol Device:R_Small_US
- added USBF1: ~, CUSTOMFOOTPRINTS:TYPE-C-SMD_HANXIA_HX-TYPE-C-6P-SY, symbol USB-C Female HX TYPE-C 6P SY:USB-C Female HX TYPE-C 6P SY
- added USBM1: ~, CUSTOMFOOTPRINTS:USB-C Male 918-118A2021Y40006, symbol USB-C Male 918-118A2021Y40006:USB-C Male 918-118A2021Y40006
- added VR_MCU1: ~, CUSTOMFOOTPRINTS:SOT-223-3_L6.5-W3.4-P2.30-LS7.0-BR, symbol SSP1117-3.3V_Voltage_Regulator:SSP1117-3.3V Voltage Regulator
- C10, C11: footprint (none) -> Resistor_SMD:R_0603_1608Metric_Pad0.98x0.95mm_HandSolder
- L2: footprint Inductor_SMD:L_0402_1005Metric -> Inductor_SMD:L_0603_1608Metric
- LPF_1: footprint footprints:DLF-4_1P6X0P8 -> CUSTOMFOOTPRINTS:LowPassFilter_DLF-4_1P6X0P8
- U3: footprint VFQFN68-8x8mm -> CUSTOMFOOTPRINTS:VFQFN68-8x8mm-L
- X1: footprint CUSTOMFOOTPRINTS:SMD1610 -> CUSTOMFOOTPRINTS:CRYSTAL-SMD_L1.6-W1.0
Connections:
- net 3.3V_PHONE: now also C17.1, Rn1.1, VR_MCU1.2 (VOUT), VR_MCU1.4 (FIN)
- net GND: now also C17.2, C18.2, C7.2, USBF1.A12 (GND), USBF1.B12 (GND), USBM1.1 (G), USBM1.16 (G), USBM1.8 (G), USBM1.9 (G), VR_MCU1.1 (ADJ/GND)
- net SERIAL_D+: now also U3.53 (PA12), Rn2.1, Rn2.2, USBM1.12 (D+), USBM1.4 (D+)
- net SERIAL_D-: now also U3.52 (PA11), Rn3.1, Rn3.2, USBM1.13 (D-), USBM1.5 (D-)
- net SMPSFB: now also C18.1
- net USB_M_IN_5V: now also C7.1, USBF1.A9 (VBUS), USBF1.B9 (VBUS), USBM1.10 (V), USBM1.15 (V), USBM1.2 (V), USBM1.7 (V), VR_MCU1.3 (VIN)
- net USB_BOOT0: now reaches U3.5 (PH3-BOOT0)
- net USB_BOOT0: now also Rn1.2
- net 3.3V_PC: no longer names the net of U3.60 (PC12)
- new net CC1: USBF1.A5 (CC1), USBM1.3 (CC1)
- new net CC2: USBF1.B5 (CC2), USBM1.11 (CC2)
- no-connect marks 20 -> 23
Other:
- note added: "16 PIN USB-C MALE RECEPTACLE"
- note added: "6 PIN FEMALE USBC RECEPTACLE"
- note added: "Either use a pad I can solder or have a tiny button/DIP switch from this trace to 3V3"
- note added: "FIN pin is usually Vout for 1117 voltage regulators"
- note added: "Pull HIGH on MCU startup to enter (usb/uart) bootloader"
- note added: "USB data pins for bootloader/flashing"
- note added: "im just gonna let these be 0603 0 ohm resistors as placeholder, i can desolder and replace with capacitors some other time if necessary"
- note removed: "Signifies we're a device requesting power with 5.1k ohms to ground"
- note removed: "do I even need to decouple this can i just rawdog it"
- note removed: "if overkill, can use voltage divider instead (cuz pc is infinite power supply anywys)"
- note removed: "ph3-boot0 is useful or no?"
- note removed: "this can be any GPIO pin really, i just sample as an input for when it's logic HIGH"
- moved on the sheet: AE1, FM1, FM2, FM3, FM4, LPF_1, M1, M2, M3, M4, U3, X1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
